File: KeyboardPCBWorkshop/KeyboardPCBWorkshop.kicad_pcb (KiCad board)
At the start: 2 copper layers, 77 x 38.1 mm, 29 parts, among them J1 AVR-ISP-6, SW1 SW_Push, SW2 SW_Push, SW3 SW_Push, SW4 SW_Push, SW5 SW_Push, U1 ATmega32U4-A, U2 PRTR5V0U2X, Y1 Crystal_GND24_Small

Commit message: FINISHED w/ERRORS?
Routing:
- net +5V: track 66.7 -> 98.1 mm, vias 2 -> 4
- net GND: track 115.2 -> 138.4 mm
- net MOSI: track 53.1 -> 32.4 mm, vias 0 -> 1
- net row1: track 55.9 -> 48.5 mm, vias 0 -> 2
- net RESET: track 37.1 -> 42.4 mm, vias 0 -> 2
- net VCC: track 27.2 -> 27.4 mm, vias 2 -> 0
- added copper zone on B.Cu, net GND
