File: KeyboardPCBWorkshop/PreGroundFill-KeyboardPCBWorkshop.kicad_pcb (KiCad board)
At the start: 2 copper layers, 77 x 38.1 mm, 29 parts, among them J1 AVR-ISP-6, SW1 SW_Push, SW2 SW_Push, SW3 SW_Push, SW4 SW_Push, SW5 SW_Push, U1 ATmega32U4-A, U2 PRTR5V0U2X, Y1 Crystal_GND24_Small

Commit message: FINISHED w/ERRORS?
Routing:
- net MOSI: track 53.1 -> 32.4 mm, vias 0 -> 1
- net row1: track 55.9 -> 48.5 mm, vias 0 -> 2
- net RESET: track 37.1 -> 42.4 mm, vias 0 -> 2
Changed lines of the file:
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@@
   (segment (start 168.6 49.475) (end 166.0125 49.475) (width 0.25) (layer "B.Cu") (net 8))
   (segment (start 171.45 52.325) (end 168.6 49.475) (width 0.25) (layer "B.Cu") (net 8))
-  (segment (start 170.7936 75.3939) (end 153.1189 75.3939) (width 0.25) (layer "B.Cu") (net 9))
-  (segment (start 152.4 74.675) (end 151.6811 75.3939) (width 0.25) (layer "B.Cu") (net 9))
-  (segment (start 153.1189 75.3939) (end 152.4 74.675) (width 0.25) (layer "B.Cu") (net 9))
-  (segment (start 132.459 69.859) (end 128.4625 65.8625) (width 0.25) (layer "B.Cu") (net 9))
-  (segment (start 139.900267 71.775) (end 135.779173 71.775) (width 0.25) (layer "B.Cu") (net 9))
-  (segment (start 128.4625 60.5375) (end 128.5375 60.4625) (width 0.25) (layer "B.Cu") (net 9))
-  (segment (start 135.511173 72.043) (end 132.795827 72.043) (width 0.25) (layer "B.Cu") (net 9))
-  (segment (start 171.45 74.7375) (end 170.7936 75.3939) (width 0.25) (layer "B.Cu") (net 9))
-  (segment (start 135.779173 71.775) (end 135.511173 72.043) (width 0.25) (layer "B.Cu") (net 9))
-  (segment (start 151.6811 75.3939) (end 142.86265 75.3939) (width 0.25) (layer "B.Cu") (net 9))
-  (segment (start 132.795827 72.043) (end 132.459 71.706173) (width 0.25) (layer "B.Cu") (net 9))
-  (segment (start 142.86265 75.3939) (end 140.6325 73.16375) (width 0.25) (layer "B.Cu") (net 9))
-  (segment (start 128.5375 60.4625) (end 129.5375 60.4625) (width 0.25) (layer "B.Cu") (net 9))
-  (segment (start 140.6325 73.16375) (end 140.6325 72.507233) (width 0.25) (layer "B.Cu") (net 9))
-  (segment (start 140.6325 72.507233) (end 139.900267 71.775) (width 0.25) (layer "B.Cu") (net 9))
-  (segment (start 132.459 71.706173) (end 132.459 69.859) (width 0.25) (layer "B.Cu") (net 9))
-  (segment (start 128.4625 65.8625) (end 128.4625 60.5375) (width 0.25) (layer "B.Cu") (net 9))
+  (segment (start 137.06475 64.29375) (end 133.223 60.452) (width 0.25) (layer "F.Cu") (net 9))
+  (segment (start 138.1125 64.29375) (end 137.06475 64.29375) (width 0.25) (layer "F.Cu") (net 9))
+  (via (at 138.1125 64.29375) (size 0.8) (drill 0.4) (layers "F.Cu" "B.Cu") (net 9))
+  (via (at 133.223 60.452) (size 0.8) (drill 0.4) (layers "F.Cu" "B.Cu") (net 9))
+  (segment (start 149.424733 74.675) (end 148.2925 73.542767) (width 0.25) (layer "B.Cu") (net 9))
+  (segment (start 148.2925 73.542767) (end 148.2925 73.30439) (width 0.25) (layer "B.Cu") (net 9))
+  (segment (start 170.7936 75.3939) (end 171.45 74.7375) (width 0.25) (layer "B.Cu") (net 9))
+  (segment (start 133.2125 60.4625) (end 129.5375 60.4625) (width 0.25) (layer "B.Cu") (net 9))
+  (segment (start 139.28186 64.29375) (end 138.1125 64.29375) (width 0.25) (layer "B.Cu") (net 9))
+  (segment (start 152.4 74.675) (end 149.424733 74.675) (width 0.25) (layer "B.Cu") (net 9))
+  (segment (start 153.1189 75.3939) (end 170.7936 75.3939) (width 0.25) (layer "B.Cu") (net 9))
+  (segment (start 152.4 74.675) (end 153.1189 75.3939) (width 0.25) (layer "B.Cu") (net 9))
+  (segment (start 148.2925 73.30439) (end 139.28186 64.29375) (width 0.25) (layer "B.Cu") (net 9))
+  (segment (start 133.223 60.452) (end 133.2125 60.4625) (width 0.25) (layer "B.Cu") (net 9))
   (segment (start 148.97 67.945) (end 147.0025 67.945) (width 0.25) (layer "B.Cu") (net 10))
   (segment (start 152.4 71.375) (end 148.97 67.945) (width 0.25) (layer "B.Cu") (net 10))
@@
   (segment (start 115.21875 58.8625) (end 118.1375 58.8625) (width 0.25) (layer "B.Cu") (net 14))
   (segment (start 107.15625 73.87425) (end 107.15625 73.81875) (width 0.25) (layer "B.Cu") (net 14))
-  (segment (start 100.2404 75.9001) (end 100.2404 51.777874) (width 0.25) (layer "B.Cu") (net 15))
-  (segment (start 119.1375 58.0625) (end 118.1375 58.0625) (width 0.25) (layer "B.Cu") (net 15))
-  (segment (start 112.896726 48.445) (end 119.2125 54.760774) (width 0.25) (layer "B.Cu") (net 15))
-  (segment (start 101.4154 77.0751) (end 100.2404 75.9001) (width 0.25) (layer "B.Cu") (net 15))
-  (segment (start 103.573274 48.445) (end 112.896726 48.445) (width 0.25) (layer "B.Cu") (net 15))
-  (segment (start 100.2404 51.777874) (end 103.573274 48.445) (width 0.25) (layer "B.Cu") (net 15))
-  (segment (start 119.2125 54.760774) (end 119.2125 57.9875) (width 0.25) (layer "B.Cu") (net 15))
-  (segment (start 119.2125 57.9875) (end 119.1375 58.0625) (width 0.25) (layer "B.Cu") (net 15))
-  (segment (start 109.838 71.905077) (end 112.568077 69.175) (width 0.25) (layer "B.Cu") (net 16))
-  (segment (start 120.6375 64.4375) (end 120.6375 55.5625) (width 0.25) (layer "B.Cu") (net 16))
+  (segment (start 101.4154 77.0751) (end 102.5904 78.2501) (width 0.25) (layer "F.Cu") (net 15))
+  (segment (start 104.442101 78.2501) (end 106.426 76.266201) (width 0.25) (layer "F.Cu") (net 15))
+  (segment (start 106.426 76.266201) (end 106.426 73.279) (width 0.25) (layer "F.Cu") (net 15))
+  (segment (start 106.426 73.279) (end 114.3 65.405) (width 0.25) (layer "F.Cu") (net 15))
+  (segment (start 114.3 65.405) (end 114.3 57.531) (width 0.25) (layer "F.Cu") (net 15))
+  (segment (start 102.5904 78.2501) (end 104.442101 78.2501) (width 0.25) (layer "F.Cu") (net 15))
+  (via (at 114.3 57.531) (size 0.8) (drill 0.4) (layers "F.Cu" "B.Cu") (net 15))
+  (segment (start 114.3 57.531) (end 116.606 57.531) (width 0.25) (layer "B.Cu") (net 15))
+  (segment (start 116.606 57.531) (end 117.1375 58.0625) (width 0.25) (layer "B.Cu") (net 15))
+  (segment (start 117.1375 58.0625) (end 118.1375 58.0625) (width 0.25) (layer "B.Cu") (net 15))
+  (segment (start 115.951 68.199) (end 115.951 54.864) (width 0.25) (layer "F.Cu") (net 16))
+  (via (at 115.951 68.199) (size 0.8) (drill 0.4) (layers "F.Cu" "B.Cu") (net 16))
+  (via (at 115.951 54.864) (size 0.8) (drill 0.4) (layers "F.Cu" "B.Cu") (net 16))
+  (segment (start 110.7125 70.64375) (end 112.18125 69.175) (width 0.25) (layer "B.Cu") (net 16))
+  (segment (start 119.29 53.34) (end 120.6375 54.6875) (width 0.25) (layer "B.Cu") (net 16))
+  (segment (start 115.951 54.737) (end 117.348 53.34) (width 0.25) (layer "B.Cu") (net 16))
+  (segment (start 117.348 53.34) (end 119.29 53.34) (width 0.25) (layer "B.Cu") (net 16))
   (segment (start 109.838 73.937) (end 109.838 80.137) (width 0.25) (layer "B.Cu") (net 16))
+  (segment (start 109.838 73.410222) (end 110.7125 72.535722) (width 0.25) (layer "B.Cu") (net 16))
   (segment (start 103.9554 79.6151) (end 109.3161 79.6151) (width 0.25) (layer "B.Cu") (net 16))
-  (segment (start 109.838 73.937) (end 109.838 71.905077) (width 0.25) (layer "B.Cu") (net 16))
-  (segment (start 112.568077 69.175) (end 115.9 69.175) (width 0.25) (layer "B.Cu") (net 16))
-  (segment (start 115.9 69.175) (end 120.6375 64.4375) (width 0.25) (layer "B.Cu") (net 16))
+  (segment (start 115.951 54.864) (end 115.951 54.737) (width 0.25) (layer "B.Cu") (net 16))
+  (segment (start 109.838 73.937) (end 109.838 73.410222) (width 0.25) (layer "B.Cu") (net 16))
+  (segment (start 110.7125 72.535722) (end 110.7125 70.64375) (width 0.25) (layer "B.Cu") (net 16))
+  (segment (start 120.6375 54.6875) (end 120.6375 55.5625) (width 0.25) (layer "B.Cu") (net 16))
+  (segment (start 114.975 69.175) (end 115.951 68.199) (width 0.25) (layer "B.Cu") (net 16))
   (segment (start 109.3161 79.6151) (end 109.838 80.137) (width 0.25) (layer "B.Cu") (net 16))
+  (segment (start 112.18125 69.175) (end 114.975 69.175) (width 0.25) (layer "B.Cu") (net 16))
   (segment (start 133.125 65.2625) (end 129.5375 65.2625) (width 0.25) (layer "B.Cu") (net 17))
   (segment (start 133.3625 65.025) (end 133.125 65.2625) (width 0.25) (layer "B.Cu") (net 17))
